File: design_files/AST1024.sch (EAGLE design)
At the start: 7 parts, among them J1 SM05B, U1 VL53L0X

Commit message: updated documentation
Parts:
- C2: value 10uF -> 4.7uF; device tinycircuits:AS-ITM-00002 -> tinycircuits:AS-ITM-00088; PARTNO (none) -> AS-ITM-00088; VALUE (none) -> 4.7uF
- J1: device tinycircuits:AS-ITM-00340 -> tinycircuits:AS-ITM-00340EDGE
- R3: value 0.0 -> 1.00K; device tinycircuits:AS-ITM-00076 -> tinycircuits:AS-ITM-00003; PARTNO (none) -> AS-ITM-00003; VALUE (none) -> 1.00K
Other:
- note added: "Hand Populated: -"
- note added: "Hand Soldered: -"
- note added: "Non Populated: -"
- note added: "Notes: -"
- note added: "Variant: Standard"
- note added: "Wireling Distance Sensor"
- note removed: "Disconnect GPIO1 if not used (R2 Optional)"
- note removed: "TOF Sensor Board"
